File: FullInterlockingPlant/FullInterlockingPlant.kicad_pcb (KiCad board)
At the start: 2 copper layers, 0 parts

Commit message: Complete FullInterlockingPlant (without CAN)
Parts:
- added C1: .1 uf, C1, F.Cu at (72.4, 116.8)
- added C2: 1uf 35V, C1V5, F.Cu at (69.8, 170.2)
- added C3: .1 uf, C1, F.Cu at (79.4, 143.5)
- added C4: 10 uf, 50V, CP_Radial_D5.0mm_P2.00mm, F.Cu at (74.9, 144.8)
- added C5: 15 uf, 50V, CP_Radial_D5.0mm_P2.00mm, F.Cu at (150.5, 152.4)
- added C6: .1 uf, C1, F.Cu at (160.7, 143.5)
- added D1: 1N4002, D3, F.Cu at (59.7, 160.0)
- added D2: 1N4002, D3, F.Cu at (77.5, 154.9)
- added IC1: MCT6H, DIP-8__300, F.Cu at (52.1, 154.9)
- added J1: RPI_GPIO, vasch_strip_20x2, F.Cu at (38.1, 143.5)
- added MH: MountingHole_2-5mm_RevA_Date21Jun2010, MountingHole_2-5mm_RevA_Date21Jun2010, F.Cu at (30.5, 111.8)
- added MH: MountingHole_2-5mm_RevA_Date21Jun2010, MountingHole_2-5mm_RevA_Date21Jun2010, F.Cu at (30.5, 175.3)
- added MH: MountingHole_2-5mm_RevA_Date21Jun2010, MountingHole_2-5mm_RevA_Date21Jun2010, F.Cu at (157.5, 111.8)
- added MH: MountingHole_2-5mm_RevA_Date21Jun2010, MountingHole_2-5mm_RevA_Date21Jun2010, F.Cu at (157.5, 175.3)
- added P1: CONN_5, ScrewTerm_2.54-5, F.Cu at (50.8, 175.3)
- added P2: CONN_5, ScrewTerm_2.54-5, F.Cu at (66.0, 175.3)
- added P3: CONN_5, ScrewTerm_2.54-5, F.Cu at (81.3, 175.3)
- added Q1: MPQ3725A, DIP-14__300, F.Cu at (53.3, 129.5)
- added Q2: MPQ2222A, DIP-14__300, F.Cu at (90.2, 161.3)
- added Q3: MPQ2222A, DIP-14__300, F.Cu at (110.5, 161.3)
- added Q4: MPQ2222A, DIP-14__300, F.Cu at (130.8, 161.3)
- added Q5: MPQ2222A, DIP-14__300, F.Cu at (151.1, 161.3)
- added Q6: MPQ2222A, DIP-14__300, F.Cu at (90.2, 125.7)
- added Q7: MPQ2222A, DIP-14__300, F.Cu at (110.5, 125.7)
- added Q8: MPQ2222A, DIP-14__300, F.Cu at (130.8, 125.7)
- added Q9: MPQ2222A, DIP-14__300, F.Cu at (151.1, 125.7)
- added R1: 10K Ohms, R1, F.Cu at (66.0, 120.7)
- added R10: 1K Ohms, R1, F.Cu at (76.2, 161.3)
- added R11: 1K Ohms, R1, F.Cu at (61.0, 153.7)
- added R12: 1K Ohms, R1, F.Cu at (45.7, 124.5)
- added R13: 1K Ohms, R1, F.Cu at (45.7, 134.6)
- added R14: 1K Ohms, R1, F.Cu at (61.0, 134.6)
- added R15: 1K Ohms, R1, F.Cu at (61.0, 124.5)
- added R16: 470 Ohms, R1, F.Cu at (45.7, 121.9)
- added R17: 470 Ohms, R1, F.Cu at (45.7, 137.2)
- added R18: 470 Ohms, R1, F.Cu at (61.0, 137.2)
- added R19: 470 Ohms, R1, F.Cu at (61.0, 121.9)
- added R2: 10K Ohms, R1, F.Cu at (66.0, 133.3)
- added R20: 1K Ohms, R1, F.Cu at (85.1, 168.9)
- added R21: 1K Ohms, R1, F.Cu at (95.2, 168.9)
- added R22: 1K Ohms, R1, F.Cu at (95.2, 153.7)
- added R23: 1K Ohms, R1, F.Cu at (85.1, 153.7)
- added R24: 150 Ohms, R1, F.Cu at (82.5, 168.9)
- added R25: 150 Ohms, R1, F.Cu at (97.8, 168.9)
- added R26: 150 Ohms, R1, F.Cu at (97.8, 153.7)
- added R27: 150 Ohms, R1, F.Cu at (82.5, 153.7)
- added R28: 1K Ohms, R1, F.Cu at (105.4, 168.9)
- added R29: 1K Ohms, R1, F.Cu at (115.6, 168.9)
- added R3: 10K Ohms, R1, F.Cu at (78.7, 135.9)
- added R30: 1K Ohms, R1, F.Cu at (115.6, 153.7)
- added R31: 1k Ohms, R1, F.Cu at (105.4, 153.7)
- added R32: 150 Ohms, R1, F.Cu at (102.9, 168.9)
- added R33: 150 Ohms, R1, F.Cu at (118.1, 168.9)
- added R34: 150 Ohms, R1, F.Cu at (118.1, 153.7)
- added R35: 150 Ohms, R1, F.Cu at (102.9, 153.7)
- added R36: 1K Ohms, R1, F.Cu at (125.7, 168.9)
- added R37: 1K Ohms, R1, F.Cu at (135.9, 168.9)
- added R38: 1K Ohms, R1, F.Cu at (135.9, 153.7)
- added R39: 1K Ohms, R1, F.Cu at (125.7, 153.7)
- added R4: 10K Ohms, R1, F.Cu at (78.7, 123.2)
- added R40: 10K Ohms, R1, F.Cu at (109.2, 135.9)
- added R41: 150 Ohms, R1, F.Cu at (123.2, 168.9)
- added R42: 150 Ohms, R1, F.Cu at (138.4, 168.9)
- added R43: 150 Ohms, R1, F.Cu at (138.4, 153.7)
- added R44: 150 Ohms, R1, F.Cu at (123.2, 153.7)
- added R45: 1K Ohms, R1, F.Cu at (146.1, 168.9)
- added R46: 1K Ohms, R1, F.Cu at (156.2, 168.9)
- added R47: 1K Ohms, R1, F.Cu at (156.2, 153.7)
- added R48: 1K Ohms, R1, F.Cu at (146.1, 153.7)
- added R49: 150 Ohms, R1, F.Cu at (143.5, 168.9)
- added R5: 270 Ohms, R1, F.Cu at (45.7, 152.4)
- added R50: 150 Ohms, R1, F.Cu at (158.8, 168.9)
- added R51: 150 Ohms, R1, F.Cu at (158.8, 153.7)
- added R52: 150 Ohms, R1, F.Cu at (143.5, 153.7)
- added R53: 1K Ohms, R1, F.Cu at (95.2, 118.1)
- added R54: 1K Ohms, R1, F.Cu at (85.1, 118.1)
- added R55: 1K Ohms, R1, F.Cu at (85.1, 133.3)
- added R56: 1K Ohms, R1, F.Cu at (95.2, 133.3)
- added R57: 150 Ohms, R1, F.Cu at (97.8, 118.1)
- added R58: 150 Ohms, R1, F.Cu at (82.5, 118.1)
- added R59: 150 Ohms, R1, F.Cu at (82.5, 133.3)
- added R6: 270 Ohms, R1, F.Cu at (45.7, 157.5)
- added R60: 150 Ohms, R1, F.Cu at (97.8, 133.3)
- added R61: 1K Ohms, R1, F.Cu at (115.6, 118.1)
- added R62: 1K Ohms, R1, F.Cu at (105.4, 118.1)
- added R63: 1K Ohms, R1, F.Cu at (105.4, 133.3)
- added R64: 1k Ohms, R1, F.Cu at (115.6, 133.3)
- added R65: 150 Ohms, R1, F.Cu at (118.1, 118.1)
- added R66: 150 Ohms, R1, F.Cu at (102.9, 118.1)
- added R67: 150 Ohms, R1, F.Cu at (102.9, 133.3)
- added R68: 150 Ohms, R1, F.Cu at (118.1, 133.3)
- added R69: 1K Ohms, R1, F.Cu at (135.9, 118.1)
- added R7: 100 Ohms, R1, F.Cu at (61.0, 148.6)
- added R70: 1K Ohms, R1, F.Cu at (125.7, 118.1)
- added R71: 1K Ohms, R1, F.Cu at (125.7, 133.3)
- added R72: 1K Ohms, R1, F.Cu at (135.9, 133.3)
- added R73: 10K Ohms, R1, F.Cu at (130.8, 151.1)
- added R74: 10K Ohms, R1, F.Cu at (121.9, 149.9)
- added R75: 150 Ohms, R1, F.Cu at (138.4, 118.1)
- added R76: 150 Ohms, R1, F.Cu at (123.2, 118.1)
- added R77: 150 Ohms, R1, F.Cu at (123.2, 133.3)
- added R78: 150 Ohms, R1, F.Cu at (138.4, 133.3)
- added R79: 1K Ohms, R1, F.Cu at (156.2, 118.1)
- added R8: 100 Ohms, R1, F.Cu at (76.2, 163.8)
- added R80: 1K Ohms, R1, F.Cu at (146.1, 118.1)
- added R81: 1K Ohms, R1, F.Cu at (146.1, 133.3)
- added R82: 1K Ohms, R1, F.Cu at (156.2, 133.3)
- added R83: 150 Ohms, R1, F.Cu at (158.8, 118.1)
- added R84: 150 Ohms, R1, F.Cu at (143.5, 118.1)
- added R85: 150 Ohms, R1, F.Cu at (143.5, 133.3)
- added R86: 150 Ohms, R1, F.Cu at (158.8, 133.3)
- added R9: 1K Ohms, R1, F.Cu at (61.0, 151.1)
- added T1: Motor 1, ScrewTerm_2.54-5, F.Cu at (50.8, 111.8)
- added T10: H3, ScrewTerm_2.54-5, F.Cu at (129.5, 111.8)
- added T11: H4, ScrewTerm_2.54-5, F.Cu at (144.8, 111.8)
- added T2: Motor 2, ScrewTerm_2.54-5, F.Cu at (66.0, 111.8)
- added T3: 12 to 16 Volts, ScrewTerm2.54-2, F.Cu at (77.5, 111.8)
- added T4: H1, ScrewTerm_2.54-5, F.Cu at (99.1, 175.3)
- added T5: H2, ScrewTerm_2.54-5, F.Cu at (114.3, 175.3)
- added T6: H3, ScrewTerm_2.54-5, F.Cu at (129.5, 175.3)
- added T7: H4, ScrewTerm_2.54-5, F.Cu at (144.8, 175.3)
- added T8: H1, ScrewTerm_2.54-5, F.Cu at (99.1, 111.8)
- added T9: H2, ScrewTerm_2.54-5, F.Cu at (114.3, 111.8)
- added U1: 74AHCT00, DIP-14__300, F.Cu at (72.4, 129.5)
- added U2: LM324N, DIP-14__300, F.Cu at (68.6, 156.2)
- added U3: MCP23017, DIP-28__300, F.Cu at (100.3, 143.5)
- added U4: MCP23017, DIP-28__300, F.Cu at (139.7, 143.5)
- added Z1: 1N5229B, D3, F.Cu at (62.2, 165.1)
Routing:
- net GND: track 0.00 -> 590.4 mm, vias 0 -> 5
- net +3.3V: track 0.00 -> 282.6 mm, vias 0 -> 3
- net +5V: track 0.00 -> 242.9 mm
- net +12V: track 0.00 -> 141.9 mm, vias 0 -> 2
- net SCL: track 0.00 -> 106.5 mm
- net SDA: track 0.00 -> 104.1 mm
- net /Quad Signals 1/GP1.1: track 0.00 -> 90.9 mm, vias 0 -> 3
- net /Quad Signals 2/GP0.5: track 0.00 -> 78.5 mm, vias 0 -> 5
- net /Quad Signals 2/GP0.3: track 0.00 -> 78.2 mm, vias 0 -> 6
- net /Quad Signals 1/GP1.4: track 0.00 -> 77.2 mm, vias 0 -> 4
- net /Quad Signals 1/GP1.6: track 0.00 -> 76.7 mm, vias 0 -> 7
- net /Quad Signals 1/GP1.0: track 0.00 -> 70.5 mm, vias 0 -> 1
- net /Quad Signals 2/GP0.4: track 0.00 -> 70.2 mm, vias 0 -> 4
- net /Quad Signals 1/GP1.7: track 0.00 -> 67.9 mm, vias 0 -> 1
- net /Quad Signals 1/GP1.3: track 0.00 -> 66.0 mm, vias 0 -> 1
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Other:
- board outline added: 137.2 x 73.7 mm
