File: FullInterlockingPlant/FullInterlockingPlant.sch (KiCad schematic (older format))
At the start: 4 parts

Commit message: Complete FullInterlockingPlant (without CAN)
Parts:
- gave numbers to parts that had none: 4
Connections:
- net labels added: VDD
Changed lines of the file:
@@
 LIBS:FullInterlockingPlant-cache
 LIBS:FullInterlockingPlant-cache
-LIBS:SMCSenseHAT-cache
 EELAYER 27 0
 EELAYER END
 $Descr A4 11693 8268
 encoding utf-8
-Sheet 1 2
+Sheet 1 4
 Title ""
 Date "13 may 2018"
@@
 $EndDescr
 $Comp
-L RPI_GPIO J?
+L RPI_GPIO J1
 U 1 1 5AF76E30
 P 1550 1250
-F 0 "J?" H 2300 1500 60  0000 C CNN
+F 0 "J1" H 2300 1500 60  0000 C CNN
 F 1 "RPI_GPIO" H 2300 1400 60  0000 C CNN
 F 2 "~" H 1550 1250 60  0000 C CNN
@@
 $EndSheet
 $Comp
-L +3.3V #PWR?
+L +3.3V #PWR01
 U 1 1 5AF7B7BF
 P 1350 1250
-F 0 "#PWR?" H 1350 1210 30  0001 C CNN
+F 0 "#PWR01" H 1350 1210 30  0001 C CNN
 F 1 "+3.3V" H 1350 1360 30  0000 C CNN
 F 2 "" H 1350 1250 60  0000 C CNN
@@
 $EndComp
 $Comp
-L +3.3V #PWR?
+L +3.3V #PWR02
 U 1 1 5AF7B7DA
 P 1350 2050
-F 0 "#PWR?" H 1350 2010 30  0001 C CNN
+F 0 "#PWR02" H 1350 2010 30  0001 C CNN
 F 1 "+3.3V" H 1350 2160 30  0000 C CNN
 F 2 "" H 1350 2050 60  0000 C CNN
@@
 $EndComp
 $Comp
-L GND #PWR?
+L GND #PWR03
 U 1 1 5AF7B7F5
 P 1350 1650
-F 0 "#PWR?" H 1350 1650 30  0001 C CNN
+F 0 "#PWR03" H 1350 1650 30  0001 C CNN
 F 1 "GND" H 1350 1580 30  0001 C CNN
 F 2 "" H 1350 1650 60  0000 C CNN
@@
 $EndComp
 $Comp
-L GND #PWR?
+L GND #PWR04
 U 1 1 5AF7B810
 P 1350 2450
-F 0 "#PWR?" H 1350 2450 30  0001 C CNN
+F 0 "#PWR04" H 1350 2450 30  0001 C CNN
 F 1 "GND" H 1350 2380 30  0001 C CNN
 F 2 "" H 1350 2450 60  0000 C CNN
@@
 $EndComp
 $Comp
-L GND #PWR?
+L GND #PWR05
 U 1 1 5AF7B837
 P 1350 3150
-F 0 "#PWR?" H 1350 3150 30  0001 C CNN
+F 0 "#PWR05" H 1350 3150 30  0001 C CNN
 F 1 "GND" H 1350 3080 30  0001 C CNN
 F 2 "" H 1350 3150 60  0000 C CNN
@@
 $EndComp
 $Comp
-L GND #PWR?
+L GND #PWR06
 U 1 1 5AF7C0AA
 P 3250 2850
-F 0 "#PWR?" H 3250 2850 30  0001 C CNN
+F 0 "#PWR06" H 3250 2850 30  0001 C CNN
 F 1 "GND" H 3250 2780 30  0001 C CNN
 F 2 "" H 3250 2850 60  0000 C CNN
@@
 $EndComp
 $Comp
-L GND #PWR?
+L GND #PWR07
 U 1 1 5AF7C0C5
 P 3250 2650
-F 0 "#PWR?" H 3250 2650 30  0001 C CNN
+F 0 "#PWR07" H 3250 2650 30  0001 C CNN
 F 1 "GND" H 3250 2580 30  0001 C CNN
 F 2 "" H 3250 2650 60  0000 C CNN
@@
 $EndComp
 $Comp
-L GND #PWR?
+L GND #PWR08
 U 1 1 5AF7C0E0
 P 3250 2150
-F 0 "#PWR?" H 3250 2150 30  0001 C CNN
+F 0 "#PWR08" H 3250 2150 30  0001 C CNN
 F 1 "GND" H 3250 2080 30  0001 C CNN
 F 2 "" H 3250 2150 60  0000 C CNN
@@
 $EndComp
 $Comp
-L GND #PWR?
+L GND #PWR09
 U 1 1 5AF7C0FB
 P 3250 1850
-F 0 "#PWR?" H 3250 1850 30  0001 C CNN
+F 0 "#PWR09" H 3250 1850 30  0001 C CNN
 F 1 "GND" H 3250 1780 30  0001 C CNN
 F 2 "" H 3250 1850 60  0000 C CNN
@@
 $EndComp
 $Comp
-L GND #PWR?
+L GND #PWR010
 U 1 1 5AF7C116
 P 3250 1450
-F 0 "#PWR?" H 3250 1450 30  0001 C CNN
+F 0 "#PWR010" H 3250 1450 30  0001 C CNN
 F 1 "GND" H 3250 1380 30  0001 C CNN
 F 2 "" H 3250 1450 60  0000 C CNN
@@
 $EndComp
 $Comp
-L +5V #PWR?
+L +5V #PWR011
 U 1 1 5AF7C1FD
 P 3250 1250
-F 0 "#PWR?" H 3250 1340 20  0001 C CNN
+F 0 "#PWR011" H 3250 1340 20  0001 C CNN
 F 1 "+5V" H 3250 1340 30  0000 C CNN
 F 2 "" H 3250 1250 60  0000 C CNN
@@
 #26
 $Comp
-L CONN_5 P?
+L CONN_5 P1
 U 1 1 5AF819CD
 P 1150 4300
-F 0 "P?" V 1100 4300 50  0000 C CNN
+F 0 "P1" V 1100 4300 50  0000 C CNN
 F 1 "CONN_5" V 1200 4300 50  0000 C CNN
 F 2 "~" H 1150 4300 60  0000 C CNN
@@
 $EndComp
 $Comp
-L CONN_5 P?
+L CONN_5 P2
 U 1 1 5AF819F4
 P 1750 4300
-F 0 "P?" V 1700 4300 50  0000 C CNN
+F 0 "P2" V 1700 4300 50  0000 C CNN
 F 1 "CONN_5" V 1800 4300 50  0000 C CNN
 F 2 "~" H 1750 4300 60  0000 C CNN
@@
 $EndComp
 $Comp
-L CONN_5 P?
+L CONN_5 P3
 U 1 1 5AF81A0F
 P 2350 4300
-F 0 "P?" V 2300 4300 50  0000 C CNN
+F 0 "P3" V 2300 4300 50  0000 C CNN
 F 1 "CONN_5" V 2400 4300 50  0000 C CNN
 F 2 "~" H 2350 4300 60  0000 C CNN
@@
 $EndComp
 $Comp
-L +3.3V #PWR?
+L +3.3V #PWR012
 U 1 1 5AF81A2A
 P 950 3900
-F 0 "#PWR?" H 950 3860 30  0001 C CNN
+F 0 "#PWR012" H 950 3860 30  0001 C CNN
 F 1 "+3.3V" H 950 4010 30  0000 C CNN
 F 2 "" H 950 3900 60  0000 C CNN
@@
 $EndComp
 $Comp
-L GND #PWR?
+L GND #PWR013
 U 1 1 5AF81B59
 P 2550 3900
-F 0 "#PWR?" H 2550 3900 30  0001 C CNN
+F 0 "#PWR013" H 2550 3900 30  0001 C CNN
 F 1 "GND" H 2550 3830 30  0001 C CNN
 F 2 "" H 2550 3900 60  0000 C CNN
@@
 Text GLabel 2450 3900 1    39   Input ~ 0
 #26
+$Sheet
+S 6350 1250 1150 1200
+U 5AF84489
+F0 "Quad Signals 1" 50
+F1 "QuadSignals1.sch" 50
+$EndSheet
+$Sheet
+S 8200 1250 1200 1200
+U 5AF844A3
+F0 "Quad Signals 2" 50
+F1 "QuadSignals2.sch" 50
+$EndSheet
+$Comp
+L VDD #PWR014
+U 1 1 5AF853F3
+P 950 2250
+F 0 "#PWR014" H 950 2350 30  0001 C CNN
+F 1 "VDD" H 950 2360 30  0000 C CNN
+F 2 "" H 950 2250 60  0000 C CNN
+F 3 "" H 950 2250 60  0000 C CNN
+	1    950  2250
+	1    0    0    -1
+$EndComp
+$Comp
+L +3.3V #PWR015
+U 1 1 5AF8540E
+P 950 2250
+F 0 "#PWR015" H 950 2210 30  0001 C CNN
+F 1 "+3.3V" H 950 2360 30  0000 C CNN
+F 2 "" H 950 2250 60  0000 C CNN
+F 3 "" H 950 2250 60  0000 C CNN
+	1    950  2250
+	-1   0    0    1
+$EndComp
 $EndSCHEMATC
