File: YardBoss/YardBoss.kicad_pcb (KiCad board)
At the start: 2 copper layers, 160 x 73.7 mm, 94 parts, among them IC1 MCT6H, IC4 MCT6H, J1 RPI_GPIO, J2 Termination, J3 RJ45, J4 RJ45, P1 CE0, P2 CE1, P3 CS, P4 I2C Expansion, P6 CONN_5, P7 CONN_5, Q1 MPQ3725A, Q4 FQU5P20TU, Q5 MPQ3725A, T1 PS1A PS1C PS1B M1A M1B, T10 12 Volts, T11 PS3A PS3C PS3B M3A M3B, T12 PS4A PS4C PS4B M4A M4B, T2 PS2A PS2C PS2B M2A M2B, U1 74AHCT00, U10 74AHCT00, U11 LM324N, U2 LM324N, U7 MCP2515, U8 MCP2551, U9 LM78S05CV, X1 16 MHz

Commit message: Complete YardBoss board.
Parts:
- added P8: + 12 Volts -, ScrewTerm2.54-2, F.Cu at (162.6, 175.3)
- C10, C8: footprint C2 -> C1
- D7, D8: value SB240-E3/54 -> SB240E
- P6: value CONN_5 -> +3.3V #5 #6 #13 #19
- P7: value CONN_5 -> #26 #16 #20 #21 GND
- T10: value 12 Volts -> - 12 Volts +
Routing:
- net GND: track 597.4 -> 66.2 mm, vias 7 -> 4
- net /Stall Motors 2/M Select 2: track 195.0 -> 117.5 mm, vias 7 -> 6
- net +5V: track 207.0 -> 275.7 mm, vias 8 -> 7
- net /Stall Motors 2/MSelect 1: track 169.8 -> 113.4 mm
- net +12V: track 318.5 -> 367.2 mm, vias 3 -> 21
- net +3.3V: track 307.1 -> 346.8 mm, vias 2 -> 12
- net SCL: track 152.0 -> 188.6 mm
- net SDA: track 159.9 -> 189.4 mm, vias 11 -> 4
- net N-00000100: track 26.0 -> 48.9 mm, vias 2 -> 4
- net /Stall Motors 2/Point Sense 2: track 143.5 -> 165.2 mm, vias 0 -> 2
- net N-00000109: track 102.1 -> 123.8 mm, vias 1 -> 5
- net /Stall Motors 1/Point Sense 2: track 102.8 -> 123.6 mm
- net N-0000099: track 19.9 -> 40.2 mm, vias 0 -> 6
- net N-0000035: track 37.5 -> 56.7 mm, vias 6 -> 3
- net /Stall Motors 1/MSelect 1: track 68.7 -> 87.8 mm, vias 5 -> 3
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- added copper zone on F.Cu, net /CAN Transciver/Heat Sink Pad
- added copper zone on B.Cu, net GND
