File: YardBoss/LEDDaughterBoard/LEDDaughterBoard.sch (KiCad schematic (older format))
At the start: 2 parts, among them J1 I2CIN, J2 I2COUT

Commit message: Complete LED daughter board (Yard Boss).
Parts:
- added C1: .1 uf, ~, symbol C
- added C2: 10 uf, ~, symbol CP1
- added C3: 15 uf, ~, symbol CP1
- added P1: 2 1 0, ~, symbol CONN_3X2
- added P2: L04 L05 L06 L07 C, ~, symbol CONN_5
- added P3: C L14 L15 L16 L17, ~, symbol CONN_5
- added P4: L00 L01 L02 L03 C, ~, symbol CONN_5
- added P5: C L13 L12 L11 L10, ~, symbol CONN_5
- added Q1, Q2, Q3, Q4: MPQ2222A, TO116, symbol MPQ2222A
- added R1, R10, R11, R12, R17, R18, R19, R2, R20, R25, R26, R27, R28, R3, R4, R9: 1K Ohms, ~, symbol R
- added R13, R14, R15, R16, R21, R22, R23, R24, R29, R30, R31, R32, R5, R6, R7, R8: 150 Ohms, ~, symbol R
- added RR1: 10K Ohms, ~, symbol RR4
- added U1: MCP23017, ~, symbol MCP23017
Connections:
- net labels added: L00, L01, L02, L03, L04, L05, L06, L07, L10, L11, L12, L13, L14, L15, L16, L17
- wire segments 14 -> 183
