File: SPILEDDriverAddOn/SPILEDDriverAddOn.kicad_pcb (KiCad board)
At the start: 2 copper layers, 125.7 x 47 mm, 17 parts, among them P1 CONN_8, P2 CONN_9, P3 CONN_9, P4 CONN_9, P5 CONN_9, U1 74HCT595N, U2 ULN2803A, U3 74HCT595N, U4 ULN2803A, U5 74HCT595N, U6 ULN2803A, U7 74HCT595N, U8 ULN2803A

Commit message: Finalized PCBs
Parts:
- added MH: MountingHole_2-5mm_RevA_Date21Jun2010, MountingHole_2-5mm_RevA_Date21Jun2010, F.Cu at (53.3, 102.9)
- added MH: MountingHole_2-5mm_RevA_Date21Jun2010, MountingHole_2-5mm_RevA_Date21Jun2010, F.Cu at (58.4, 142.2)
- added MH: MountingHole_2-5mm_RevA_Date21Jun2010, MountingHole_2-5mm_RevA_Date21Jun2010, F.Cu at (170.2, 142.2)
- added MH: MountingHole_2-5mm_RevA_Date21Jun2010, MountingHole_2-5mm_RevA_Date21Jun2010, F.Cu at (170.2, 123.2)
- P1: value CONN_8 -> SPI Expansion
- P2, P3, P4, P5: value CONN_9 -> 0 1 2 3 4 5 6 7 D +; footprint ScrewTerm_2.54-9 -> ScrewTerm_2.54-10
- moved P2 1.27 mm to (71.1, 101.6)
- moved P3 1.27 mm to (99.1, 101.6)
- moved P4 1.27 mm to (127.0, 101.6)
- moved P5 1.27 mm to (154.9, 101.6)
Routing:
- net N-0000094: track 10.2 -> 8.89 mm
- net N-0000091: track 10.2 -> 8.89 mm
- net N-0000090: track 10.2 -> 8.89 mm
- net N-0000089: track 10.2 -> 8.89 mm
- net N-0000088: track 10.2 -> 8.89 mm
- net N-0000087: track 10.2 -> 8.89 mm
- net N-0000086: track 10.2 -> 8.89 mm
- net N-0000085: track 10.2 -> 8.89 mm
- net N-0000070: track 10.2 -> 8.89 mm
- net N-0000067: track 10.2 -> 8.89 mm
- net N-0000066: track 10.2 -> 8.89 mm
- net N-0000065: track 10.2 -> 8.89 mm
- net N-0000064: track 10.2 -> 8.89 mm
- net N-0000063: track 10.2 -> 8.89 mm
- net N-0000062: track 10.2 -> 8.89 mm
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Other:
- board text added: "Port F"
- board text added: "Port G"
- board text added: "Port H"
- board text added: "Port I"
