File: ESP32QuadOCDect/ESP32QuadOCDect.sch (KiCad schematic (older format))
At the start: 2 parts, among them U0 ESP32_DEVKIT_C or TTGO-T1

Commit message: Started work on ESP32 boards.
Connections:
- wire segments 7 -> 9
Changed lines of the file:
@@
 F0 "CAN Transceiver" 50
 F1 "CAN_Transeiver.sch" 50
+F2 "CAN_TX" I L 4300 2000 60
+F3 "CAN_RX" I L 4300 2150 60
 $EndSheet
 $Sheet
@@
 F1 "PowerSupply.sch" 50
 $EndSheet
+Wire Wire Line
+	4300 2000 3550 2000
+Wire Wire Line
+	4300 2150 3550 2150
 $EndSCHEMATC

Commit message: Completed design for ESP32QuadOCDect.
Connections:
- net labels added: OD 1, OD 2, OD 3, OD 4
Changed lines of the file:
@@
 LIBS:sn65hvd233-ht
 LIBS:lm2574n-5
+LIBS:mct6h
+LIBS:bridge
 LIBS:ESP32QuadOCDect-cache
 EELAYER 27 0
@@
 $Descr A4 11693 8268
 encoding utf-8
-Sheet 1 3
+Sheet 1 7
 Title ""
-Date "8 mar 2019"
+Date "9 mar 2019"
 Rev ""
 Comp ""
@@
 Wire Wire Line
 	4300 2150 3550 2150
+$Sheet
+S 1850 4050 1750 1700
+U 5C70A8FB
+F0 "Occupancy Detector 1" 50
+F1 "OD1.sch" 50
+F2 "OD1" O L 1850 4250 60
+$EndSheet
+$Sheet
+S 4400 4050 1750 1700
+U 5C831BA4
+F0 "Occupancy Detector 2" 50
+F1 "OD2.sch" 50
+F2 "OD2" O L 4400 4350 60
+$EndSheet
+$Sheet
+S 6850 4150 1850 1850
+U 5C831BA3
+F0 "Occupancy Detector 3" 50
+F1 "OD3.sch" 50
+F2 "OD3" O L 6850 4400 60
+$EndSheet
+$Sheet
+S 9400 4200 1600 1800
+U 5C831BA2
+F0 "Occupancy Detector 4" 50
+F1 "OD4.sch" 50
+F2 "OD4" O L 9400 4400 60
+$EndSheet
+Text Label 2650 2000 2    25   ~ 0
+OD 1
+Text Label 2650 2050 2    25   ~ 0
+OD 2
+Text Label 2650 1650 2    25   ~ 0
+OD 3
+Text Label 2650 1700 2    25   ~ 0
+OD 4
+Text Label 1850 4250 2    25   ~ 0
+OD 1
+Text Label 4400 4350 2    25   ~ 0
+OD 2
+Text Label 6850 4400 2    25   ~ 0
+OD 3
+Text Label 9400 4400 2    25   ~ 0
+OD 4
 $EndSCHEMATC
