File: ESP32BaseBoard/ESP32BaseBoard.sch (KiCad schematic (older format))
At the start: 2 parts, among them U0 ESP32_DEVKIT_C or TTGO-T1

Commit message: Started work on ESP32 boards.
Connections:
- wire segments 7 -> 13
Changed lines of the file:
@@
 F0 "CAN Transceiver" 50
 F1 "CAN_Transeiver.sch" 50
+F2 "CAN_TX" I L 4300 1850 60
+F3 "CAN_RX" I L 4300 2050 60
 $EndSheet
 $Sheet
@@
 F1 "PowerSupply.sch" 50
 $EndSheet
+Wire Wire Line
+	4300 1850 4100 1850
+Wire Wire Line
+	4100 1850 4100 2000
+Wire Wire Line
+	4100 2000 3550 2000
+Wire Wire Line
+	3550 2150 4200 2150
+Wire Wire Line
+	4200 2150 4200 2050
+Wire Wire Line
+	4200 2050 4300 2050
 $EndSCHEMATC

Commit message: Spec. parts for CAN tranciver, Power Supply.
Parts:
- JP0: Mouser Part Number (none) -> dummp
- U0: Mouser Part Number (none) -> dummy
Changed lines of the file:
@@
 Sheet 1 3
 Title ""
-Date "8 mar 2019"
+Date "16 mar 2019"
 Rev ""
 Comp ""
@@
 F 2 "~" H 3100 2000 60  0000 C CNN
 F 3 "~" H 3100 2000 60  0000 C CNN
+F 4 "dummy" H 3100 2000 60  0001 C CNN "Mouser Part Number"
 	1    3100 2000
 	1    0    0    -1
@@
 F 2 "~" H 3750 1850 60  0000 C CNN
 F 3 "~" H 3750 1850 60  0000 C CNN
+F 4 "dummp" H 3750 1850 60  0001 C CNN "Mouser Part Number"
 	1    3750 1850
 	1    0    0    -1
