File: ESP32BaseBoard/PowerSupply.sch (KiCad schematic (older format))
At the start: 5 parts, among them U3 LM2574N-5.0

Commit message: Spec. parts for CAN tranciver, Power Supply.
Parts:
- C4: Mouser Part Number (none) -> 140-REA221M1EBK0811P
- C5: Mouser Part Number (none) -> 140-REA220M2ABK0811P
- D3: Mouser Part Number (none) -> 625-SB160-E3
- L1: Mouser Part Number (none) -> PE-52627NL
- U3: Mouser Part Number (none) -> 926-LM2574N-5.0/NOPB
Changed lines of the file:
@@
 Sheet 3 3
 Title ""
-Date "8 mar 2019"
+Date "16 mar 2019"
 Rev ""
 Comp ""
@@
 F 2 "~" H 5200 2800 60  0000 C CNN
 F 3 "~" H 5200 2800 60  0000 C CNN
+F 4 "926-LM2574N-5.0/NOPB" H 5200 2800 60  0001 C CNN "Mouser Part Number"
 	1    5200 2800
 	1    0    0    -1
@@
 F 2 "~" H 5950 2900 60  0000 C CNN
 F 3 "~" H 5950 2900 60  0000 C CNN
+F 4 "140-REA220M2ABK0811P" H 5950 2900 60  0001 C CNN "Mouser Part Number"
 	1    5950 2900
 	1    0    0    -1
@@
 F 2 "~" H 3700 2800 60  0000 C CNN
 F 3 "~" H 3700 2800 60  0000 C CNN
+F 4 "140-REA221M1EBK0811P" H 3700 2800 60  0001 C CNN "Mouser Part Number"
 	1    3700 2800
 	1    0    0    -1
@@
 F 2 "~" H 4550 2900 60  0000 C CNN
 F 3 "~" H 4550 2900 60  0000 C CNN
+F 4 "PE-52627NL" H 4550 2900 60  0001 C CNN "Mouser Part Number"
 	1    4550 2900
 	1    0    0    -1
@@
 F 2 "~" H 4850 3100 60  0000 C CNN
 F 3 "~" H 4850 3100 60  0000 C CNN
+F 4 "625-SB160-E3" H 4850 3100 60  0001 C CNN "Mouser Part Number"
 	1    4850 3100
 	0    -1   -1   0
