File: ESP32-HalfSiding/CAN_Transeiver.sch (KiCad schematic (older format))
At the start: 14 parts, among them J1 RJ45, J2 RJ45, T1 + 15 in -, T2 + 15 out -, U1 TCAN332DR, U2 SN65HVD233-HT

Commit message: ESP32-HalfSiding updates
Parts:
- C1, C3: symbol C -> C-RESCUE-ESP32-HalfSiding
- C2: symbol CP1 -> CP1-RESCUE-ESP32-HalfSiding
- R1, R2: symbol R -> R-RESCUE-ESP32-HalfSiding
Changed lines of the file:
@@
 EESchema Schematic File Version 2
+LIBS:ESP32-HalfSiding-rescue
 LIBS:power
 LIBS:device
@@
 LIBS:memory
 LIBS:xilinx
-LIBS:special
 LIBS:microcontrollers
 LIBS:dsp
@@
 LIBS:bridge
 LIBS:ESP32-HalfSiding-cache
-EELAYER 27 0
+EELAYER 25 0
 EELAYER END
 $Descr A4 11693 8268
@@
 $EndComp
 $Comp
-L GND #PWR013
+L GND-RESCUE-ESP32-HalfSiding #PWR013
 U 1 1 5C828CBC
 P 4100 3800
@@
 $EndComp
 $Comp
-L GND #PWR014
+L GND-RESCUE-ESP32-HalfSiding #PWR014
 U 1 1 5C828CCB
 P 4100 4950
@@
 Connection ~ 3750 4400
 $Comp
-L C C1
+L C-RESCUE-ESP32-HalfSiding C1
 U 1 1 5C828DA1
 P 4650 3800
@@
 $EndComp
 $Comp
-L CP1 C2
+L CP1-RESCUE-ESP32-HalfSiding C2
 U 1 1 5C828DB0
 P 5000 3800
@@
 CANL
 $Comp
-L R R1
+L R-RESCUE-ESP32-HalfSiding R1
 U 1 1 5C828F93
 P 5850 3650
@@
 $EndComp
 $Comp
-L R R2
+L R-RESCUE-ESP32-HalfSiding R2
 U 1 1 5C828FA2
 P 6550 3650
@@
 	6700 4150 6600 4150
 $Comp
-L C C3
+L C-RESCUE-ESP32-HalfSiding C3
 U 1 1 5C8290C3
 P 6200 4750
@@
 $EndComp
 $Comp
-L GND #PWR015
+L GND-RESCUE-ESP32-HalfSiding #PWR015
 U 1 1 5C8290D2
 P 6200 5100
@@
 	7450 3000 7450 5050
 $Comp
-L GND #PWR016
+L GND-RESCUE-ESP32-HalfSiding #PWR016
 U 1 1 5C8295F7
 P 6750 2650
