File: ESP32-HalfSiding/drivers.sch (KiCad schematic (older format))
At the start: 14 parts, among them P1 0 1 2, P2 C A0 A1 A2 A3 A4 A5 A6 A7, P3 C B0 B1 B2 B3 B4 B5 B6 B7, U4 MCP23017, U5 TBD62X83A, U6 TBD62X83A

Commit message: ESP32-HalfSiding updates
Parts:
- C6: symbol C -> C-RESCUE-ESP32-HalfSiding
- U4: symbol MCP23017 -> MCP23017-RESCUE-ESP32-HalfSiding
Changed lines of the file:
@@
 EESchema Schematic File Version 2
+LIBS:ESP32-HalfSiding-rescue
 LIBS:power
 LIBS:device
@@
 LIBS:memory
 LIBS:xilinx
-LIBS:special
 LIBS:microcontrollers
 LIBS:dsp
@@
 LIBS:bridge
 LIBS:ESP32-HalfSiding-cache
-EELAYER 27 0
+EELAYER 25 0
 EELAYER END
 $Descr A4 11693 8268
@@
 $EndDescr
 $Comp
-L MCP23017 U4
+L MCP23017-RESCUE-ESP32-HalfSiding U4
 U 1 1 5C73ECE1
 P 4950 2400
@@
 	9750 5300 9750 5250
 $Comp
-L GND #PWR021
+L GND-RESCUE-ESP32-HalfSiding #PWR021
 U 1 1 5C73ECFB
 P 9050 1150
@@
 	8550 1100 8550 1000
 $Comp
-L GND #PWR022
+L GND-RESCUE-ESP32-HalfSiding #PWR022
 U 1 1 5C73ECFD
 P 8550 5450
@@
 $EndComp
 $Comp
-L GND #PWR024
+L GND-RESCUE-ESP32-HalfSiding #PWR024
 U 1 1 5C73ECFF
 P 4850 3800
@@
 Connection ~ 4950 1150
 $Comp
-L C C6
+L C-RESCUE-ESP32-HalfSiding C6
 U 1 1 5C73ED06
 P 5600 1150
@@
 	5300 950  5600 950
 $Comp
-L GND #PWR025
+L GND-RESCUE-ESP32-HalfSiding #PWR025
 U 1 1 5C73ED07
 P 5600 1400
@@
 	5600 1350 5600 1400
 $Comp
-L GND #PWR026
+L GND-RESCUE-ESP32-HalfSiding #PWR026
 U 1 1 5C73ED09
 P 6900 1250
@@
 	6400 950  6400 1150
 $Comp
-L GND #PWR027
+L GND-RESCUE-ESP32-HalfSiding #PWR027
 U 1 1 5C73ED0A
 P 6400 5450
@@
 $EndComp
 $Comp
-L GND #PWR032
+L GND-RESCUE-ESP32-HalfSiding #PWR032
 U 1 1 5C7402B8
 P 3100 2200
