File: ESP32-MultiFunction/StallMotors4.sch (KiCad schematic (older format))
At the start: 13 parts, among them U2 74HCT00, U4 74HCT00, U5 TC4428, U6 TC4428, U7 TC4428, U8 TC4428

Commit message: Restore broken files.
Parts:
- C6, C7: symbol ESP32-MultiFunction-rescue:C_Small -> C_Small
- RR1: symbol ESP32-MultiFunction-rescue:4814P-2 -> 4814P-2
- Term1, Term2, Term3, Term4: symbol ESP32-MultiFunction-rescue:Screw_Terminal_01x05 -> Screw_Terminal_01x05
- U2, U4: symbol ESP32-MultiFunction-rescue:74HCT00 -> 74HCT00
- U5, U6, U7, U8: symbol ESP32-MultiFunction-rescue:TC4428 -> TC4428
Changed lines of the file:
@@
-EESchema Schematic File Version 4
+EESchema Schematic File Version 2
+LIBS:power
+LIBS:device
+LIBS:switches
+LIBS:relays
+LIBS:motors
+LIBS:transistors
+LIBS:conn
+LIBS:linear
+LIBS:regul
+LIBS:74xx
+LIBS:cmos4000
+LIBS:adc-dac
+LIBS:memory
+LIBS:xilinx
+LIBS:microcontrollers
+LIBS:dsp
+LIBS:microchip
+LIBS:analog_switches
+LIBS:motorola
+LIBS:texas
+LIBS:intel
+LIBS:audio
+LIBS:interface
+LIBS:digital-audio
+LIBS:philips
+LIBS:display
+LIBS:cypress
+LIBS:siliconi
+LIBS:opto
+LIBS:atmel
+LIBS:contrib
+LIBS:esp32_devboards
+LIBS:sn65hvd233-ht
+LIBS:lm2574n-5
+LIBS:MCP23xxx
+LIBS:tbd62x83a
+LIBS:tc442x
+LIBS:mct6h
+LIBS:bridge
+LIBS:pca9685
+LIBS:4814p-2
+LIBS:mechanical
+LIBS:graphic_symbols
+LIBS:references
 LIBS:ESP32-MultiFunction-cache
-EELAYER 30 0
+EELAYER 25 0
 EELAYER END
 $Descr A4 11693 8268
@@
 $EndDescr
 $Comp
-L ESP32-MultiFunction-rescue:74HCT00 U2
+L 74HCT00 U2
 U 2 1 60CD31DC
 P 2000 1900
@@
 $EndComp
 $Comp
-L ESP32-MultiFunction-rescue:74HCT00 U2
+L 74HCT00 U2
 U 3 1 60CD3211
 P 2000 2700
@@
 $EndComp
 $Comp
-L ESP32-MultiFunction-rescue:74HCT00 U2
+L 74HCT00 U2
 U 4 1 60CD324F
 P 2000 3400
@@
 $EndComp
 $Comp
-L ESP32-MultiFunction-rescue:74HCT00 U4
+L 74HCT00 U4
 U 1 1 60CD3BDA
 P 2050 4600
@@
 $EndComp
 $Comp
-L ESP32-MultiFunction-rescue:74HCT00 U4
+L 74HCT00 U4
 U 2 1 60CD3BE0
 P 2050 5300
@@
 $EndComp
 $Comp
-L ESP32-MultiFunction-rescue:74HCT00 U4
+L 74HCT00 U4
 U 3 1 60CD3BE6
 P 2050 6100
@@
 $EndComp
 $Comp
-L ESP32-MultiFunction-rescue:74HCT00 U4
+L 74HCT00 U4
 U 4 1 60CD3BEC
 P 2050 6800
@@
 $EndComp
 $Comp
-L ESP32-MultiFunction-rescue:4814P-2 RR1
+L 4814P-2 RR1
 U 1 1 60CD4592
 P 900 4200
@@
 $EndComp
 $Comp
-L ESP32-MultiFunction-rescue:C_Small C6
+L C_Small C6
 U 1 1 60CD54EA
 P 2850 950
@@
 $EndComp
 $Comp
-L ESP32-MultiFunction-rescue:C_Small C7
+L C_Small C7
 U 1 1 60CD553D
 P 3200 950
@@
 $EndComp
 $Comp
-L ESP32-MultiFunction-rescue:TC4428 U5
+L TC4428 U5
 U 1 1 60CD5772
 P 4250 1100
@@
 $EndComp
 $Comp
-L ESP32-MultiFunction-rescue:TC4428 U5
+L TC4428 U5
 U 2 1 60CD57A9
 P 4250 1900
@@
 $EndComp
 $Comp
-L ESP32-MultiFunction-rescue:TC4428 U6
+L TC4428 U6
 U 1 1 60CD593C
 P 4250 2700
@@
 $EndComp
 $Comp
-L ESP32-MultiFunction-rescue:TC4428 U6
+L TC4428 U6
 U 2 1 60CD5AD3
 P 4250 3500
@@
 $EndComp
 $Comp
-L ESP32-MultiFunction-rescue:TC4428 U7
+L TC4428 U7
 U 1 1 60CD5B99
 P 7400 1100
@@
 $EndComp
 $Comp
-L ESP32-MultiFunction-rescue:TC4428 U7
+L TC4428 U7
 U 2 1 60CD5DFA
 P 7400 1900
@@
 $EndComp
 $Comp
-L ESP32-MultiFunction-rescue:TC4428 U8
+L TC4428 U8
 U 1 1 60CD5F16
 P 7400 2700
@@
 $EndComp
 $Comp
-L ESP32-MultiFunction-rescue:TC4428 U8
+L TC4428 U8
 U 2 1 60CD5F79
 P 7400 3500
@@
 $EndComp
 $Comp
-L ESP32-MultiFunction-rescue:Screw_Terminal_01x05 Term1
+L Screw_Terminal_01x05 Term1
 U 1 1 60CF9376
 P 10000 1000
@@
 $EndComp
 $Comp
-L ESP32-MultiFunction-rescue:Screw_Terminal_01x05 Term2
+L Screw_Terminal_01x05 Term2
 U 1 1 60CD6A61
 P 10000 1800
@@
 $EndComp
 $Comp
-L ESP32-MultiFunction-rescue:Screw_Terminal_01x05 Term3
+L Screw_Terminal_01x05 Term3
 U 1 1 60CD6B08
 P 10000 2650
@@
 $EndComp
 $Comp
-L ESP32-MultiFunction-rescue:Screw_Terminal_01x05 Term4
+L Screw_Terminal_01x05 Term4
 U 1 1 60CD6C75
 P 10000 3600
@@
 $EndComp
 $Comp
-L ESP32-MultiFunction-rescue:+3V3 #PWR036
+L +3V3 #PWR036
 U 1 1 60CD8400
 P 1800 750
@@
 $EndComp
 $Comp
-L ESP32-MultiFunction-rescue:+3V3 #PWR037
+L +3V3 #PWR037
 U 1 1 60CD84B5
 P 1800 4200
@@
 $EndComp
 $Comp
-L ESP32-MultiFunction-rescue:GND #PWR038
+L GND #PWR038
 U 1 1 60CD85AF
 P 1800 3800
@@
 $EndComp
 $Comp
-L ESP32-MultiFunction-rescue:GND #PWR039
+L GND #PWR039
 U 1 1 60CD86EE
 P 1850 7200
@@
 	1800 750  1800 1000
 $Comp
-L ESP32-MultiFunction-rescue:74HCT00 U2
+L 74HCT00 U2
 U 1 1 60CD316F
 P 2000 1200
@@
 	3200 1050 2850 1050
 $Comp
-L ESP32-MultiFunction-rescue:GND #PWR040
+L GND #PWR040
 U 1 1 60CD9FDD
 P 3200 1200
@@
 Motor4
 $Comp
-L ESP32-MultiFunction-rescue:GND #PWR041
+L GND #PWR041
 U 1 1 60CDE058
 P 4500 2150
@@
 $EndComp
 $Comp
-L ESP32-MultiFunction-rescue:GND #PWR042
+L GND #PWR042
 U 1 1 60CDE09A
 P 7600 2150
@@
 $EndComp
 $Comp
-L ESP32-MultiFunction-rescue:GND #PWR043
+L GND #PWR043
 U 1 1 60CDE17D
 P 4450 3750
@@
 $EndComp
 $Comp
-L ESP32-MultiFunction-rescue:GND #PWR044
+L GND #PWR044
 U 1 1 60CDE1BF
 P 7700 3750
@@
 $EndComp
 $Comp
-L ESP32-MultiFunction-rescue:+12V #PWR045
+L +12V #PWR045
 U 1 1 60CDE3F5
 P 4500 850
-AR Path="/60CDE3F5" Ref="#PWR045"  Part="1"
-AR Path="/60CD422F/60CDE3F5" Ref="#PWR045"  Part="1"
 F 0 "#PWR045" H 4500 700 50  0001 C CNN
 F 1 "+12V" H 4500 990 50  0000 C CNN
@@
 $EndComp
 $Comp
-L ESP32-MultiFunction-rescue:+12V #PWR046
+L +12V #PWR046
 U 1 1 60CDE437
 P 7600 900
-AR Path="/60CDE437" Ref="#PWR046"  Part="1"
-AR Path="/60CD422F/60CDE437" Ref="#PWR046"  Part="1"
 F 0 "#PWR046" H 7600 750 50  0001 C CNN
 F 1 "+12V" H 7600 1040 50  0000 C CNN
@@
 $EndComp
 $Comp
-L ESP32-MultiFunction-rescue:+12V #PWR047
+L +12V #PWR047
 U 1 1 60CDE58D
 P 7750 2450
-AR Path="/60CDE58D" Ref="#PWR047"  Part="1"
-AR Path="/60CD422F/60CDE58D" Ref="#PWR047"  Part="1"
 F 0 "#PWR047" H 7750 2300 50  0001 C CNN
 F 1 "+12V" H 7750 2590 50  0000 C CNN
@@
 $EndComp
 $Comp
-L ESP32-MultiFunction-rescue:+12V #PWR048
+L +12V #PWR048
 U 1 1 60CDE691
 P 4650 2500
-AR Path="/60CDE691" Ref="#PWR048"  Part="1"
-AR Path="/60CD422F/60CDE691" Ref="#PWR048"  Part="1"
 F 0 "#PWR048" H 4650 2350 50  0001 C CNN
 F 1 "+12V" H 4650 2640 50  0000 C CNN
@@
 	4500 2100 4500 2150
 $Comp
-L ESP32-MultiFunction-rescue:GND #PWR049
+L GND #PWR049
 U 1 1 60CDF082
 P 9650 3700
@@
 $EndComp
 $Comp
-L ESP32-MultiFunction-rescue:GND #PWR050
+L GND #PWR050
 U 1 1 60CDF132
 P 9650 2750
@@
 $EndComp
 $Comp
-L ESP32-MultiFunction-rescue:GND #PWR051
+L GND #PWR051
 U 1 1 60CDF3BC
 P 9700 1900
@@
 $EndComp
 $Comp
-L ESP32-MultiFunction-rescue:GND #PWR052
+L GND #PWR052
 U 1 1 60CDF400
 P 9700 1100
