File: ESP32-S3-MultiFunction/OccDetect4.sch (KiCad schematic (older format))
At the start: 35 parts, among them U601 LM339, U602 LM339

Commit message: Finalize part numbers.
Parts:
- Term601: Mouser Part Number 651-1725711 -> 651-1725711
Changed lines of the file:
@@
 F 2 "Connectors_Terminal_Blocks:TerminalBlock_Pheonix_MPT-2.54mm_8pol" H 800 3450 50  0001 C CNN
 F 3 "" H 800 3450 50  0001 C CNN
-F 4 " 651-1725711" H 800 3450 60  0001 C CNN "Mouser Part Number"
+F 4 "651-1725711" H 800 3450 60  0001 C CNN "Mouser Part Number"
 	1    800  3450
 	-1   0    0    -1
