File: LPC176x_MultiFunction/Buttons.sch (KiCad schematic (older format))
At the start: 31 parts

Commit message: Nearing completion of LPC176x_MultiFunction.
Parts:
- Term901: renamed from Term?; value 1 2 3 4 5 6 7 8 GND -> GND 8 7 6 5 4 3 2 1
- gave numbers to parts that had none: 20
Connections:
- net Button1: now also U902.6; no longer U902.2
- net Button2: now also U902.8; no longer U902.4
- net Button3: now also U902.10; no longer U902.6
- net Button4: now also U902.12; no longer U902.8
- net Button5: now also U901.6; no longer U901.2
- net Button6: now also U901.8; no longer U901.4
- net Button7: now also U901.10; no longer U901.6
- net Button8: now also U901.12; no longer U901.8
- net GND: now also U901.1, U901.3, U902.1, U902.3; no longer U901.11, U901.13, U902.11, U902.13
- net at C907.1, R905.2, Term901.1 (Pin_1): now also U902.5; no longer U902.1
- net at C908.1, R906.2, Term901.2 (Pin_2): now also U902.9; no longer U902.3
- net at C910.1, R908.2, Term901.3 (Pin_3): now also U902.11; no longer U902.5
- net at C909.1, R907.2, Term901.4 (Pin_4): now also U902.13; no longer U902.9
- net at C904.1, R903.2, Term901.5 (Pin_5): now also U901.5; no longer U901.1
- net at C905.1, R904.2, Term901.6 (Pin_6): now also U901.9; no longer U901.3
- net at C902.1, R901.2, Term901.7 (Pin_7): now also U901.11; no longer U901.5
- net at C903.1, R902.2, Term901.8 (Pin_8): now also U901.13; no longer U901.9
