File: LPC176x_MultiFunction/LEDDrivers.sch (KiCad schematic (older format))
At the start: 25 parts

Commit message: Nearing completion of LPC176x_MultiFunction.
Parts:
- Term801: renamed from Term?; value +V 1 2 3 4 5 6 7 8 GND -> GND 8 7 6 5 4 3 2 1 +
- gave numbers to parts that had none: 20
Connections:
- net LED1: now also U801.4 (IN); no longer U801.2 (IN)
- net LED2: now also U801.2 (IN); no longer U801.4 (IN)
- net LED3: now also U802.4 (IN); no longer U802.2 (IN)
- net LED4: now also U802.2 (IN); no longer U802.4 (IN)
- net LED5: now also U803.4 (IN); no longer U803.2 (IN)
- net LED6: now also U803.2 (IN); no longer U803.4 (IN)
- net LED7: now also U804.4 (IN); no longer U804.2 (IN)
- net LED8: now also U804.2 (IN); no longer U804.4 (IN)
- net at R805.2, R806.2: now also U802.5 (Out); no longer U802.7 (Out)
- net at R807.2, R808.2: now also U802.7 (Out); no longer U802.5 (Out)
- net at R801.2, R802.2: now also U801.5 (Out); no longer U801.7 (Out)
- net at R803.2, R804.2: now also U801.7 (Out); no longer U801.5 (Out)
- net at R813.2, R814.2: now also U804.5 (Out); no longer U804.7 (Out)
- net at R815.2, R816.2: now also U804.7 (Out); no longer U804.5 (Out)
- net at R809.2, R810.2: now also U803.5 (Out); no longer U803.7 (Out)
- net at R811.2, R812.2: now also U803.7 (Out); no longer U803.5 (Out)
Changed lines of the file:
@@
 LIBS:4814p-2
 LIBS:tc442x
+LIBS:pca9685
+LIBS:tbd62x83a
+LIBS:mechanical
 LIBS:LPC176x_MultiFunction-cache
 EELAYER 25 0
@@
 $Descr USLetter 11000 8500
 encoding utf-8
-Sheet 8 9
+Sheet 8 11
 Title "ESP32 S3 Multifunction Board"
 Date ""
@@
 $EndDescr
 $Comp
-L TC4426 U?
-U 1 1 632FBBDD
+L TC4426 U802
+U 2 1 632FBBDD
 P 2625 2900
-F 0 "U?" H 2625 2600 60  0000 C CNN
+F 0 "U802" H 2625 2600 60  0000 C CNN
 F 1 "TC4426" H 2625 3200 60  0000 C CNN
 F 2 "Housings_SOIC:SOIC-8_3.9x4.9mm_Pitch1.27mm" H 2625 2900 60  0001 C CNN
 F 3 "" H 2625 2900 60  0000 C CNN
 F 4 "579-TC1426COA713" H 2625 2900 60  0001 C CNN "Mouser Part Number"
-	1    2625 2900
-	1    0    0    -1
-$EndComp
-$Comp
-L TC4426 U?
-U 2 1 632FBBDE
+	2    2625 2900
+	1    0    0    -1
+$EndComp
+$Comp
+L TC4426 U802
+U 1 1 632FBBDE
 P 2625 3750
-F 0 "U?" H 2625 3450 60  0000 C CNN
+F 0 "U802" H 2625 3450 60  0000 C CNN
 F 1 "TC4426" H 2625 4050 60  0000 C CNN
 F 2 "Housings_SOIC:SOIC-8_3.9x4.9mm_Pitch1.27mm" H 2625 3750 60  0001 C CNN
 F 3 "" H 2625 3750 60  0000 C CNN
 F 4 "579-TC1426COA713" H 2625 3750 60  0001 C CNN "Mouser Part Number"
-	2    2625 3750
-	1    0    0    -1
-$EndComp
-$Comp
-L R R?
+	1    2625 3750
+	1    0    0    -1
+$EndComp
+$Comp
+L R R802
 U 1 1 632FBBDF
 P 3825 1300
-F 0 "R?" V 3905 1300 50  0000 C CNN
+F 0 "R802" V 3905 1300 50  0000 C CNN
 F 1 "1.5K Ohms" V 3825 1300 50  0000 C CNN
 F 2 "Resistors_SMD:R_0603" V 3755 1300 50  0001 C CNN
@@
 $EndComp
 $Comp
-L R R?
+L R R801
 U 1 1 632FBBE0
 P 3825 1150
-F 0 "R?" V 3905 1150 50  0000 C CNN
+F 0 "R801" V 3905 1150 50  0000 C CNN
 F 1 "R" V 3825 1150 50  0000 C CNN
 F 2 "Resistors_THT:R_Axial_DIN0207_L6.3mm_D2.5mm_P7.62mm_Horizontal" V 3755 1150 50  0001 C CNN
@@
 $EndComp
 $Comp
-L R R?
+L R R804
 U 1 1 632FBBE1
 P 3825 2100
-F 0 "R?" V 3905 2100 50  0000 C CNN
+F 0 "R804" V 3905 2100 50  0000 C CNN
 F 1 "1.5K Ohms" V 3825 2100 50  0000 C CNN
 F 2 "Resistors_SMD:R_0603" V 3755 2100 50  0001 C CNN
@@
 $EndComp
 $Comp
-L R R?
+L R R803
 U 1 1 632FBBE2
 P 3825 1950
-F 0 "R?" V 3905 1950 50  0000 C CNN
+F 0 "R803" V 3905 1950 50  0000 C CNN
 F 1 "R" V 3825 1950 50  0000 C CNN
 F 2 "Resistors_THT:R_Axial_DIN0207_L6.3mm_D2.5mm_P7.62mm_Horizontal" V 3755 1950 50  0001 C CNN
@@
 $EndComp
 $Comp
-L R R?
+L R R806
 U 1 1 632FBBE3
 P 3825 2900
-F 0 "R?" V 3905 2900 50  0000 C CNN
+F 0 "R806" V 3905 2900 50  0000 C CNN
 F 1 "1.5K Ohms" V 3825 2900 50  0000 C CNN
 F 2 "Resistors_SMD:R_0603" V 3755 2900 50  0001 C CNN
@@
 $EndComp
 $Comp
-L R R?
+L R R805
 U 1 1 632FBBE4
 P 3825 2750
-F 0 "R?" V 3905 2750 50  0000 C CNN
+F 0 "R805" V 3905 2750 50  0000 C CNN
 F 1 "R" V 3825 2750 50  0000 C CNN
 F 2 "Resistors_THT:R_Axial_DIN0207_L6.3mm_D2.5mm_P7.62mm_Horizontal" V 3755 2750 50  0001 C CNN
@@
 $EndComp
 $Comp
-L R R?
+L R R808
 U 1 1 632FBBE5
 P 3825 3750
-F 0 "R?" V 3905 3750 50  0000 C CNN
+F 0 "R808" V 3905 3750 50  0000 C CNN
 F 1 "1.5K Ohms" V 3825 3750 50  0000 C CNN
 F 2 "Resistors_SMD:R_0603" V 3755 3750 50  0001 C CNN
@@
 $EndComp
 $Comp
-L R R?
+L R R807
 U 1 1 632FBBE6
 P 3825 3600
-F 0 "R?" V 3905 3600 50  0000 C CNN
+F 0 "R807" V 3905 3600 50  0000 C CNN
 F 1 "R" V 3825 3600 50  0000 C CNN
 F 2 "Resistors_THT:R_Axial_DIN0207_L6.3mm_D2.5mm_P7.62mm_Horizontal" V 3755 3600 50  0001 C CNN
@@
 $EndComp
 $Comp
-L Screw_Terminal_01x10 Term?
+L Screw_Terminal_01x10 Term801
 U 1 1 632FBBE7
 P 5225 3000
-F 0 "Term?" H 5275 3550 50  0000 C CNN
-F 1 "+V 1 2 3 4 5 6 7 8 GND" V 5425 2875 50  0000 C CNN
+F 0 "Term801" H 5275 3550 50  0000 C CNN
+F 1 "GND 8 7 6 5 4 3 2 1 +" V 5425 2875 50  0000 C CNN
 F 2 "Connectors_Terminal_Blocks:TerminalBlock_Pheonix_MPT-2.54mm_10pol" H 5225 3000 50  0001 C CNN
 F 3 "" H 5225 3000 50  0001 C CNN
@@
 $EndComp
 $Comp
-L GND #PWR?
+L GND #PWR079
 U 1 1 632FBBE8
 P 5025 3625
-F 0 "#PWR?" H 5025 3375 50  0001 C CNN
+F 0 "#PWR079" H 5025 3375 50  0001 C CNN
 F 1 "GND" H 5025 3475 50  0000 C CNN
 F 2 "" H 5025 3625 50  0001 C CNN
@@
 LED4
 $Comp
-L TC4426 U?
-U 1 1 632FBC04
+L TC4426 U801
+U 2 1 632FBC04
 P 2575 1300
-F 0 "U?" H 2575 1000 60  0000 C CNN
+F 0 "U801" H 2575 1000 60  0000 C CNN
 F 1 "TC4426" H 2575 1600 60  0000 C CNN
 F 2 "Housings_SOIC:SOIC-8_3.9x4.9mm_Pitch1.27mm" H 2575 1300 60  0001 C CNN
 F 3 "" H 2575 1300 60  0000 C CNN
 F 4 "579-TC1426COA713" H 2575 1300 60  0001 C CNN "Mouser Part Number"
-	1    2575 1300
-	1    0    0    -1
-$EndComp
-$Comp
-L TC4426 U?
-U 2 1 632FBC05
+	2    2575 1300
+	1    0    0    -1
+$EndComp
+$Comp
+L TC4426 U801
+U 1 1 632FBC05
 P 2575 2100
-F 0 "U?" H 2575 1800 60  0000 C CNN
+F 0 "U801" H 2575 1800 60  0000 C CNN
 F 1 "TC4426" H 2575 2400 60  0000 C CNN
 F 2 "Housings_SOIC:SOIC-8_3.9x4.9mm_Pitch1.27mm" H 2575 2100 60  0001 C CNN
 F 3 "" H 2575 2100 60  0000 C CNN
 F 4 "579-TC1426COA713" H 2575 2100 60  0001 C CNN "Mouser Part Number"
-	2    2575 2100
-	1    0    0    -1
-$EndComp
-$Comp
-L GND #PWR?
+	1    2575 2100
+	1    0    0    -1
+$EndComp
+$Comp
+L GND #PWR080
 U 1 1 632FBC06
 P 2525 2450
-F 0 "#PWR?" H 2525 2200 50  0001 C CNN
+F 0 "#PWR080" H 2525 2200 50  0001 C CNN
 F 1 "GND" H 2525 2300 50  0000 C CNN
 F 2 "" H 2525 2450 50  0001 C CNN
@@
 $EndComp
 $Comp
-L GND #PWR?
+L GND #PWR081
 U 1 1 632FBC07
 P 2575 4200
-F 0 "#PWR?" H 2575 3950 50  0001 C CNN
+F 0 "#PWR081" H 2575 3950 50  0001 C CNN
 F 1 "GND" H 2575 4050 50  0000 C CNN
 F 2 "" H 2575 4200 50  0001 C CNN
@@
 LEDPower
 $Comp
-L TC4426 U?
-U 1 1 632FD544
+L TC4426 U804
+U 2 1 632FD544
 P 2750 6325
-F 0 "U?" H 2750 6025 60  0000 C CNN
+F 0 "U804" H 2750 6025 60  0000 C CNN
 F 1 "TC4426" H 2750 6625 60  0000 C CNN
 F 2 "Housings_SOIC:SOIC-8_3.9x4.9mm_Pitch1.27mm" H 2750 6325 60  0001 C CNN
 F 3 "" H 2750 6325 60  0000 C CNN
 F 4 "579-TC1426COA713" H 2750 6325 60  0001 C CNN "Mouser Part Number"
-	1    2750 6325
-	1    0    0    -1
-$EndComp
-$Comp
-L TC4426 U?
-U 2 1 632FD54B
+	2    2750 6325
+	1    0    0    -1
+$EndComp
+$Comp
+L TC4426 U804
+U 1 1 632FD54B
 P 2750 7175
-F 0 "U?" H 2750 6875 60  0000 C CNN
+F 0 "U804" H 2750 6875 60  0000 C CNN
 F 1 "TC4426" H 2750 7475 60  0000 C CNN
 F 2 "Housings_SOIC:SOIC-8_3.9x4.9mm_Pitch1.27mm" H 2750 7175 60  0001 C CNN
 F 3 "" H 2750 7175 60  0000 C CNN
 F 4 "579-TC1426COA713" H 2750 7175 60  0001 C CNN "Mouser Part Number"
-	2    2750 7175
-	1    0    0    -1
-$EndComp
-$Comp
-L R R?
+	1    2750 7175
+	1    0    0    -1
+$EndComp
+$Comp
+L R R810
 U 1 1 632FD552
 P 3950 4725
-F 0 "R?" V 4030 4725 50  0000 C CNN
+F 0 "R810" V 4030 4725 50  0000 C CNN
 F 1 "1.5K Ohms" V 3950 4725 50  0000 C CNN
 F 2 "Resistors_SMD:R_0603" V 3880 4725 50  0001 C CNN
@@
 $EndComp
 $Comp
-L R R?
+L R R809
 U 1 1 632FD558
 P 3950 4575
-F 0 "R?" V 4030 4575 50  0000 C CNN
+F 0 "R809" V 4030 4575 50  0000 C CNN
 F 1 "R" V 3950 4575 50  0000 C CNN
 F 2 "Resistors_THT:R_Axial_DIN0207_L6.3mm_D2.5mm_P7.62mm_Horizontal" V 3880 4575 50  0001 C CNN
@@
 $EndComp
 $Comp
-L R R?
+L R R812
 U 1 1 632FD55F
 P 3950 5525
-F 0 "R?" V 4030 5525 50  0000 C CNN
+F 0 "R812" V 4030 5525 50  0000 C CNN
 F 1 "1.5K Ohms" V 3950 5525 50  0000 C CNN
 F 2 "Resistors_SMD:R_0603" V 3880 5525 50  0001 C CNN
@@
 $EndComp
 $Comp
-L R R?
+L R R811
 U 1 1 632FD565
 P 3950 5375
-F 0 "R?" V 4030 5375 50  0000 C CNN
+F 0 "R811" V 4030 5375 50  0000 C CNN
 F 1 "R" V 3950 5375 50  0000 C CNN
 F 2 "Resistors_THT:R_Axial_DIN0207_L6.3mm_D2.5mm_P7.62mm_Horizontal" V 3880 5375 50  0001 C CNN
@@
 $EndComp
 $Comp
-L R R?
+L R R814
 U 1 1 632FD56C
 P 3950 6325
-F 0 "R?" V 4030 6325 50  0000 C CNN
+F 0 "R814" V 4030 6325 50  0000 C CNN
 F 1 "1.5K Ohms" V 3950 6325 50  0000 C CNN
 F 2 "Resistors_SMD:R_0603" V 3880 6325 50  0001 C CNN
@@
 $EndComp
 $Comp
-L R R?
+L R R813
 U 1 1 632FD572
 P 3950 6175
-F 0 "R?" V 4030 6175 50  0000 C CNN
+F 0 "R813" V 4030 6175 50  0000 C CNN
 F 1 "R" V 3950 6175 50  0000 C CNN
 F 2 "Resistors_THT:R_Axial_DIN0207_L6.3mm_D2.5mm_P7.62mm_Horizontal" V 3880 6175 50  0001 C CNN
@@
 $EndComp
 $Comp
-L R R?
+L R R816
 U 1 1 632FD579
 P 3950 7175
-F 0 "R?" V 4030 7175 50  0000 C CNN
+F 0 "R816" V 4030 7175 50  0000 C CNN
 F 1 "1.5K Ohms" V 3950 7175 50  0000 C CNN
 F 2 "Resistors_SMD:R_0603" V 3880 7175 50  0001 C CNN
@@
 $EndComp
 $Comp
-L R R?
+L R R815
 U 1 1 632FD57F
 P 3950 7025
-F 0 "R?" V 4030 7025 50  0000 C CNN
+F 0 "R815" V 4030 7025 50  0000 C CNN
 F 1 "R" V 3950 7025 50  0000 C CNN
 F 2 "Resistors_THT:R_Axial_DIN0207_L6.3mm_D2.5mm_P7.62mm_Horizontal" V 3880 7025 50  0001 C CNN
@@
 LED8
 $Comp
-L TC4426 U?
-U 1 1 632FD58A
+L TC4426 U803
+U 2 1 632FD58A
 P 2700 4725
-F 0 "U?" H 2700 4425 60  0000 C CNN
+F 0 "U803" H 2700 4425 60  0000 C CNN
 F 1 "TC4426" H 2700 5025 60  0000 C CNN
 F 2 "Housings_SOIC:SOIC-8_3.9x4.9mm_Pitch1.27mm" H 2700 4725 60  0001 C CNN
 F 3 "" H 2700 4725 60  0000 C CNN
 F 4 "579-TC1426COA713" H 2700 4725 60  0001 C CNN "Mouser Part Number"
-	1    2700 4725
-	1    0    0    -1
-$EndComp
-$Comp
-L TC4426 U?
-U 2 1 632FD591
+	2    2700 4725
+	1    0    0    -1
+$EndComp
+$Comp
+L TC4426 U803
+U 1 1 632FD591
 P 2700 5525
-F 0 "U?" H 2700 5225 60  0000 C CNN
+F 0 "U803" H 2700 5225 60  0000 C CNN
 F 1 "TC4426" H 2700 5825 60  0000 C CNN
 F 2 "Housings_SOIC:SOIC-8_3.9x4.9mm_Pitch1.27mm" H 2700 5525 60  0001 C CNN
 F 3 "" H 2700 5525 60  0000 C CNN
 F 4 "579-TC1426COA713" H 2700 5525 60  0001 C CNN "Mouser Part Number"
-	2    2700 5525
-	1    0    0    -1
-$EndComp
-$Comp
-L GND #PWR?
+	1    2700 5525
+	1    0    0    -1
+$EndComp
+$Comp
+L GND #PWR082
 U 1 1 632FD597
 P 2650 5875
-F 0 "#PWR?" H 2650 5625 50  0001 C CNN
+F 0 "#PWR082" H 2650 5625 50  0001 C CNN
 F 1 "GND" H 2650 5725 50  0000 C CNN
 F 2 "" H 2650 5875 50  0001 C CNN
@@
 Connection ~ 3500 4500
 $Comp
-L GND #PWR?
+L GND #PWR083
 U 1 1 632FF3CD
 P 2700 7625
-F 0 "#PWR?" H 2700 7375 50  0001 C CNN
+F 0 "#PWR083" H 2700 7375 50  0001 C CNN
 F 1 "GND" H 2700 7475 50  0000 C CNN
 F 2 "" H 2700 7625 50  0001 C CNN
