File: TTGO-T1-Booster/FANControl.sch (KiCad schematic (older format))
At the start: 7 parts

Commit message: Nearly complete: TTGO-T1-Booster.
Parts:
- gave numbers to parts that had none: 7
Changed lines of the file:
@@
 $EndDescr
 $Comp
-L Conn_01x02 J?
+L Conn_01x02 J501
 U 1 1 63B5FC89
 P 5800 2600
-F 0 "J?" H 5800 2700 50  0000 C CNN
+F 0 "J501" H 5800 2700 50  0000 C CNN
 F 1 "- Fan +" H 5800 2400 50  0000 C CNN
 F 2 "Pin_Headers:Pin_Header_Straight_1x02_Pitch2.54mm" H 5800 2600 50  0001 C CNN
@@
 $EndComp
 $Comp
-L R R?
+L R R501
 U 1 1 63B5FC8A
 P 4600 3300
-F 0 "R?" V 4680 3300 50  0000 C CNN
+F 0 "R501" V 4680 3300 50  0000 C CNN
 F 1 "1K" V 4600 3300 50  0000 C CNN
 F 2 "Resistors_SMD:R_0603" V 4530 3300 50  0001 C CNN
@@
 $EndComp
 $Comp
-L +3.3V #PWR?
+L +3.3V #PWR023
 U 1 1 63B5FC8B
 P 3450 3850
-F 0 "#PWR?" H 3450 3700 50  0001 C CNN
+F 0 "#PWR023" H 3450 3700 50  0001 C CNN
 F 1 "+3.3V" H 3450 3990 50  0000 C CNN
 F 2 "" H 3450 3850 50  0001 C CNN
@@
 $EndComp
 $Comp
-L GND #PWR?
+L GND #PWR024
 U 1 1 63B5FC8C
 P 5550 3750
-F 0 "#PWR?" H 5550 3500 50  0001 C CNN
+F 0 "#PWR024" H 5550 3500 50  0001 C CNN
 F 1 "GND" H 5550 3600 50  0000 C CNN
 F 2 "" H 5550 3750 50  0001 C CNN
@@
 $EndComp
 $Comp
-L GND #PWR?
+L GND #PWR025
 U 1 1 63B5FC8D
 P 3450 4900
-F 0 "#PWR?" H 3450 4650 50  0001 C CNN
+F 0 "#PWR025" H 3450 4650 50  0001 C CNN
 F 1 "GND" H 3450 4750 50  0000 C CNN
 F 2 "" H 3450 4900 50  0001 C CNN
@@
 TEMP_SENSE
 $Comp
-L Q_NPN_Darlington_BCEC Q?
+L Q_NPN_Darlington_BCEC Q501
 U 1 1 63B5FC8E
 P 5450 3300
-F 0 "Q?" H 5670 3350 50  0000 L CNN
+F 0 "Q501" H 5670 3350 50  0000 L CNN
 F 1 "BSP52T3G" H 5670 3250 50  0000 L CNN
 F 2 "TO_SOT_Packages_SMD:SOT-223" H 5650 3400 50  0001 C CNN
@@
 $EndComp
 $Comp
-L D D?
+L D D501
 U 1 1 63B5FC8F
 P 6100 3300
-F 0 "D?" H 6100 3400 50  0000 C CNN
+F 0 "D501" H 6100 3400 50  0000 C CNN
 F 1 "1SS352H3F" H 6100 3200 50  0000 C CNN
 F 2 "Diodes_SMD:D_SOD-323" H 6100 3300 50  0001 C CNN
@@
 	6100 3500 6100 3450
 $Comp
-L Fan_IEC60617 M?
+L Fan_IEC60617 M501
 U 1 1 63B5FC90
 P 7950 2900
-F 0 "M?" H 8100 3050 50  0000 L CNN
+F 0 "M501" H 8100 3050 50  0000 L CNN
 F 1 "Fan_IEC60617" H 8100 3000 50  0000 L TNN
 F 2 "FAN:25mmFanMount" H 8000 2760 50  0001 L CNN
@@
 $EndComp
 $Comp
-L CP1_Small C?
+L CP1_Small C501
 U 1 1 63B5FC91
 P 2300 4350
-F 0 "C?" H 2310 4420 50  0000 L CNN
+F 0 "C501" H 2310 4420 50  0000 L CNN
 F 1 "100 uf" H 2310 4270 50  0000 L CNN
 F 2 "Capacitors_SMD:C_0603" H 2300 4350 50  0001 C CNN
@@
 	4350 4500 4650 4500
 $Comp
-L MCP9700T-E_LT U?
+L MCP9700T-E_LT U501
 U 1 1 63B5FC92
 P 4350 4300
-F 0 "U?" H 4900 4250 50  0000 L CNN
+F 0 "U501" H 4900 4250 50  0000 L CNN
 F 1 "MCP9700T-E_LT" H 5050 3950 50  0000 L CNN
 F 2 "SOT65P210X110-5N:SOT65P210X110-5N" H 5300 4400 50  0001 L CNN
